File: hardware/leds.kicad_sch (KiCad schematic)
At the start: 55 parts, among them J10 Conn_01x02, J11 Conn_01x02, J12 Conn_01x02, J13 Conn_01x02, J4 Conn_01x02, J5 Conn_01x02, J6 Conn_01x02, J7 Conn_01x02, J8 Conn_01x02, J9 Conn_01x02, Q1 AO3400A, Q10 AO3400A, Q2 AO3400A, Q3 AO3400A, Q4 AO3400A, Q5 AO3400A, Q6 AO3400A, Q7 AO3400A, Q8 AO3400A, Q9 AO3400A, U4 PCA9685PW,118

Commit message: more layout and fixing OOS items
Parts:
- C11, C28, C29, C30, C31, C32, C33, C34, C35, C36, C37: symbol Device:C -> emf_beacon_ibrary:C
- C16: symbol Device:C_Polarized -> emf_beacon_ibrary:C_Polarized
- J10, J11, J12, J13, J4, J5, J6, J7, J8, J9: symbol Connector_Generic:Conn_01x02 -> emf_beacon_ibrary:Conn_01x02
- Q1, Q10, Q2, Q3, Q4, Q5, Q6, Q7, Q8, Q9: symbol Transistor_FET:AO3400A -> emf_beacon_ibrary:AO3400A
- R14, R15, R16, R17, R18, R19, R20, R21, R22, R23, R24, R25, R44, R45, R46, R47, R48, R49, R50, R51, R52, R9: symbol Device:R -> emf_beacon_ibrary:R
- U4: symbol Driver_LED:PCA9685PW -> emf_beacon_ibrary:PCA9685PW
Changed lines of the file:
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@@
 	)
 	(symbol
-		(lib_id "Connector_Generic:Conn_01x02")
+		(lib_id "emf_beacon_ibrary:Conn_01x02")
 		(at 262.89 115.57 0)
 		(unit 1)
@@
 	)
 	(symbol
-		(lib_id "Device:C")
+		(lib_id "emf_beacon_ibrary:C")
 		(at 222.25 121.92 90)
 		(unit 1)
@@
 	)
 	(symbol
-		(lib_id "Device:R")
+		(lib_id "emf_beacon_ibrary:R")
 		(at 232.41 114.3 270)
 		(unit 1)
@@
 		)
 		(property "Value" "+6V5"
-			(at 257.81 25.3999 0)
+			(at 255.27 21.59 0)
 			(effects
 				(font
 					(size 1.27 1.27)
 				)
-				(justify left)
 			)
 		)
@@
 	)
 	(symbol
-		(lib_id "Device:R")
+		(lib_id "emf_beacon_ibrary:R")
 		(at 92.71 107.95 90)
 		(unit 1)
@@
 	)
 	(symbol
-		(lib_id "Transistor_FET:AO3400A")
+		(lib_id "emf_beacon_ibrary:AO3400A")
 		(at 114.3 67.31 0)
 		(unit 1)
@@
 	)
 	(symbol
-		(lib_id "Device:C")
+		(lib_id "emf_beacon_ibrary:C")
 		(at 222.25 53.34 90)
 		(unit 1)
@@
 	)
 	(symbol
-		(lib_id "Device:R")
+		(lib_id "emf_beacon_ibrary:R")
 		(at 92.71 67.31 90)
 		(unit 1)
@@
 	)
 	(symbol
-		(lib_id "Device:R")
+		(lib_id "emf_beacon_ibrary:R")
 		(at 27.94 72.39 0)
 		(unit 1)
@@
 	)
 	(symbol
-		(lib_id "Transistor_FET:AO3400A")
+		(lib_id "emf_beacon_ibrary:AO3400A")
 		(at 195.58 148.59 0)
 		(unit 1)
@@
 	)
 	(symbol
-		(lib_id "Device:R")
+		(lib_id "emf_beacon_ibrary:R")
 		(at 232.41 99.06 270)
 		(unit 1)
@@
 	)
 	(symbol
-		(lib_id "Device:C")
+		(lib_id "emf_beacon_ibrary:C")
 		(at 222.25 83.82 90)
 		(unit 1)
@@
 	)
 	(symbol
-		(lib_id "Device:R")
+		(lib_id "emf_beacon_ibrary:R")
 		(at 92.71 77.47 90)
 		(unit 1)
@@
 	)
 	(symbol
-		(lib_id "Transistor_FET:AO3400A")
+		(lib_id "emf_beacon_ibrary:AO3400A")
 		(at 185.42 138.43 0)
 		(unit 1)
@@
 	)
 	(symbol
-		(lib_id "Device:R")
+		(lib_id "emf_beacon_ibrary:R")
 		(at 92.71 87.63 90)
 		(unit 1)
@@
 	)
 	(symbol
-		(lib_id "Device:C")
+		(lib_id "emf_beacon_ibrary:C")
 		(at 222.25 91.44 90)
 		(unit 1)
@@
 	)
 	(symbol
-		(lib_id "Transistor_FET:AO3400A")
+		(lib_id "emf_beacon_ibrary:AO3400A")
 		(at 134.62 87.63 0)
 		(unit 1)
@@
 	)
 	(symbol
-		(lib_id "Device:C")
+		(lib_id "emf_beacon_ibrary:C")
 		(at 222.25 106.68 90)
 		(unit 1)
@@
 	)
 	(symbol
-		(lib_id "Transistor_FET:AO3400A")
+		(lib_id "emf_beacon_ibrary:AO3400A")
 		(at 154.94 107.95 0)
 		(unit 1)
@@
 	)
 	(symbol
-		(lib_id "Transistor_FET:AO3400A")
+		(lib_id "emf_beacon_ibrary:AO3400A")
 		(at 104.14 57.15 0)
 		(unit 1)
@@
 	)
 	(symbol
-		(lib_id "Driver_LED:PCA9685PW")
+		(lib_id "emf_beacon_ibrary:PCA9685PW")
 		(at 50.8 96.52 0)
 		(unit 1)
@@
 	)
 	(symbol
-		(lib_id "Device:R")
+		(lib_id "emf_beacon_ibrary:R")
 		(at 232.41 83.82 270)
 		(unit 1)
@@
 	)
 	(symbol
-		(lib_id "Device:C")
+		(lib_id "emf_beacon_ibrary:C")
 		(at 222.25 68.58 90)
 		(unit 1)
@@
 	)
 	(symbol
-		(lib_id "Connector_Generic:Conn_01x02")
+		(lib_id "emf_beacon_ibrary:Conn_01x02")
 		(at 262.89 92.71 0)
 		(unit 1)
@@
 	)
 	(symbol
-		(lib_id "Connector_Generic:Conn_01x02")
+		(lib_id "emf_beacon_ibrary:Conn_01x02")
 		(at 262.89 107.95 0)
 		(unit 1)
@@
 	)
 	(symbol
-		(lib_id "Connector_Generic:Conn_01x02")
+		(lib_id "emf_beacon_ibrary:Conn_01x02")
 		(at 262.89 69.85 0)
 		(unit 1)
@@
 	)
 	(symbol
-		(lib_id "Device:R")
+		(lib_id "emf_beacon_ibrary:R")
 		(at 232.41 53.34 270)
 		(unit 1)
@@
 	)
 	(symbol
-		(lib_id "Device:R")
+		(lib_id "emf_beacon_ibrary:R")
 		(at 232.41 76.2 270)
 		(unit 1)
@@
 	)
 	(symbol
-		(lib_id "Transistor_FET:AO3400A")
+		(lib_id "emf_beacon_ibrary:AO3400A")
 		(at 175.26 128.27 0)
 		(unit 1)
@@
 	)
 	(symbol
-		(lib_id "Connector_Generic:Conn_01x02")
+		(lib_id "emf_beacon_ibrary:Conn_01x02")
 		(at 262.89 46.99 0)
 		(unit 1)
@@
 	)
 	(symbol
-		(lib_id "Connector_Generic:Conn_01x02")
+		(lib_id "emf_beacon_ibrary:Conn_01x02")
 		(at 262.89 54.61 0)
 		(unit 1)
@@
 	)
 	(symbol
-		(lib_id "Device:R")
+		(lib_id "emf_beacon_ibrary:R")
 		(at 92.71 138.43 90)
 		(unit 1)
@@
 	)
 	(symbol
-		(lib_id "Device:C")
+		(lib_id "emf_beacon_ibrary:C")
 		(at 222.25 114.3 90)
 		(unit 1)
@@
 	)
 	(symbol
-		(lib_id "Connector_Generic:Conn_01x02")
+		(lib_id "emf_beacon_ibrary:Conn_01x02")
 		(at 262.89 85.09 0)
 		(unit 1)
@@
 	)
 	(symbol
-		(lib_id "Device:C")
+		(lib_id "emf_beacon_ibrary:C")
 		(at 222.25 60.96 90)
 		(unit 1)
@@
 	)
 	(symbol
-		(lib_id "Transistor_FET:AO3400A")
+		(lib_id "emf_beacon_ibrary:AO3400A")
 		(at 144.78 97.79 0)
 		(unit 1)
@@
 	)
 	(symbol
-		(lib_id "Device:R")
+		(lib_id "emf_beacon_ibrary:R")
 		(at 232.41 60.96 270)
 		(unit 1)
@@
 	)
 	(symbol
-		(lib_id "Device:C")
+		(lib_id "emf_beacon_ibrary:C")
 		(at 222.25 99.06 90)
 		(unit 1)
@@
 	)
 	(symbol
-		(lib_id "Device:R")
+		(lib_id "emf_beacon_ibrary:R")
 		(at 92.71 148.59 90)
 		(unit 1)
@@
 	)
 	(symbol
-		(lib_id "Device:R")
+		(lib_id "emf_beacon_ibrary:R")
 		(at 232.41 91.44 270)
 		(unit 1)
@@
 	)
 	(symbol
-		(lib_id "Connector_Generic:Conn_01x02")
+		(lib_id "emf_beacon_ibrary:Conn_01x02")
 		(at 262.89 62.23 0)
 		(unit 1)
@@
 	)
 	(symbol
-		(lib_id "Device:R")
+		(lib_id "emf_beacon_ibrary:R")
 		(at 92.71 57.15 90)
 		(unit 1)
@@
 	)
 	(symbol
-		(lib_id "Device:R")
+		(lib_id "emf_beacon_ibrary:R")
 		(at 232.41 121.92 270)
 		(unit 1)
@@
 	)
 	(symbol
-		(lib_id "Transistor_FET:AO3400A")
+		(lib_id "emf_beacon_ibrary:AO3400A")
 		(at 124.46 77.47 0)
 		(unit 1)
@@
 	)
 	(symbol
-		(lib_id "Device:R")
+		(lib_id "emf_beacon_ibrary:R")
 		(at 232.41 68.58 270)
 		(unit 1)
@@
 	)
 	(symbol
-		(lib_id "Device:C_Polarized")
+		(lib_id "emf_beacon_ibrary:C_Polarized")
 		(at 250.19 35.56 0)
 		(mirror y)
@@
 	)
 	(symbol
-		(lib_id "Connector_Generic:Conn_01x02")
+		(lib_id "emf_beacon_ibrary:Conn_01x02")
 		(at 262.89 77.47 0)
 		(unit 1)
@@
 	)
 	(symbol
-		(lib_id "Device:C")
+		(lib_id "emf_beacon_ibrary:C")
 		(at 44.45 68.58 90)
 		(unit 1)
@@
 	)
 	(symbol
-		(lib_id "Device:R")
+		(lib_id "emf_beacon_ibrary:R")
 		(at 232.41 106.68 270)
 		(unit 1)
@@
 	)
 	(symbol
-		(lib_id "Transistor_FET:AO3400A")
+		(lib_id "emf_beacon_ibrary:AO3400A")
 		(at 165.1 118.11 0)
 		(unit 1)
@@
 	)
 	(symbol
-		(lib_id "Connector_Generic:Conn_01x02")
+		(lib_id "emf_beacon_ibrary:Conn_01x02")
 		(at 262.89 100.33 0)
 		(unit 1)
@@
 	)
 	(symbol
-		(lib_id "Device:R")
+		(lib_id "emf_beacon_ibrary:R")
 		(at 30.48 95.25 0)
 		(mirror y)
@@
 	)
 	(symbol
-		(lib_id "Device:C")
+		(lib_id "emf_beacon_ibrary:C")
 		(at 222.25 76.2 90)
 		(unit 1)
@@
 	)
 	(symbol
-		(lib_id "Device:R")
+		(lib_id "emf_beacon_ibrary:R")
 		(at 92.71 97.79 90)
 		(unit 1)
@@
 	)
 	(symbol
-		(lib_id "Device:R")
+		(lib_id "emf_beacon_ibrary:R")
 		(at 92.71 118.11 90)
 		(unit 1)
@@
 	)
 	(symbol
-		(lib_id "Device:R")
+		(lib_id "emf_beacon_ibrary:R")
 		(at 92.71 128.27 90)
 		(unit 1)
