File: hardware/emf_beacon.kicad_sch (KiCad schematic)
At the start: 4 parts

Commit message: preparing for release
Other:
- title: (none) -> LED Beacon
Changed lines of the file:
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@@
 	(paper "A4")
 	(title_block
-		(date "2026-04-10")
-		(rev "0")
+		(title "LED Beacon")
+		(date "2026-06-05")
+		(rev "1")
 		(company "Wires & Bits")
 	)
